File: hardware/inferface-modules/USB-2/USB-2.kicad_pcb (KiCad board)
At the start: 4 copper layers, 18 parts, among them J1 USB_device, J2 USB_B_Micro, J3 Base_Board_Interface, U1 TPD2E2U06QDBZRQ1

Commit message: Update log
Parts:
- moved U1 8.02 mm to (137.0, 79.0), turned to -90 degrees
- moved D+TP1 5.00 mm to (136.0, 94.5)
- moved D-TP1 4.27 mm to (138.0, 94.5)
- moved R1 3.91 mm to (136.0, 99.5)
- moved R2 2.99 mm to (138.0, 99.5), turned to -90 degrees
- moved J2 1.39 mm to (137.1, 108.9)
- moved TP1 1.39 mm to (130.6, 107.5)
Routing:
- net /D+: track 0.00 -> 22.0 mm
- net /D-: track 0.00 -> 21.9 mm
